File: schematic/irda-transceiver.kicad_pcb (KiCad board)
At the start: 2 copper layers, 60 x 40 mm, 32 parts, among them J1 Conn_01x03_Pin, J2 Conn_01x03_Pin, J3 Conn_01x03_Pin, J4 Conn_01x03_Pin, J5 Conn_01x03_Pin, J6 Conn_01x03_Pin, J7 Conn_01x06_Pin, U1 MCP2120-I/P, U2 TFDU4101-TT3, Y1 7.3728 MHz

Commit message: TFDU4101 transceiver updated to side view variant (TR3) instead of top view variant (TT3)
Parts:
- U2: value TFDU4101-TT3 -> TFDU4101-TR3; footprint StockLib:TFDU4101-TT3 -> StockLib:TFDU4101-TR3
Routing:
- net Net-(U1-RXIR): track 54.2 -> 27.7 mm
- net Net-(J5-Pin_2): track 31.8 -> 50.2 mm
- net Net-(U2-VCC2/IRED_AN): track 32.7 -> 39.5 mm
- net Net-(D1-K): track 22.1 -> 17.4 mm
- net Net-(J4-Pin_2): track 48.0 -> 44.7 mm
- net VCC: track 122.6 -> 121.4 mm
Other:
- board text added: "0"
- board text added: "1"
- board text added: "IRDA TRANSCEIVER MODULE V1.1"
- board text added: "TFDU4101 TR3"
- board text removed: "IRDA TRANSCEIVER MODULE V1.0"
- board text removed: "TFDU4101"
