File: schematic/irda-transceiver.kicad_pcb (KiCad board)
At the start: 2 copper layers, 60 x 40 mm, 32 parts, among them J1 Conn_01x03_Pin, J2 Conn_01x03_Pin, J3 Conn_01x03_Pin, J4 Conn_01x03_Pin, J5 Conn_01x03_Pin, J6 Conn_01x03_Pin, J7 Conn_01x06_Pin, U1 MCP2120-I/P, U2 TFDU4101-TR3, Y1 7.3728 MHz

Commit message: PCB traces refined
Routing:
- net Net-(J6-Pin_2): track 36.6 -> 37.2 mm
Changed lines of the file:
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@@
+	)
+	(segment
+		(start 36.4379 9.3041)
+		(end 31.518 14.224)
+		(width 0.2)
+		(layer "B.Cu")
+		(net 5)
+	)
+	(segment
+		(start 31.518 14.224)
+		(end 29.5497 14.224)
+		(width 0.2)
+		(layer "B.Cu")
+		(net 5)
+	)
+	(segment
+		(start 29.5497 14.224)
+		(end 28.5337 15.24)
+		(width 0.2)
+		(layer "B.Cu")
+		(net 5)
+	)
+	(segment
+		(start 28.5337 15.24)
+		(end 27.432 15.24)
+		(width 0.2)
+		(layer "B.Cu")
+		(net 5)
+	)
+	(segment
+		(start 41.9318 11.7058)
+		(end 39.5301 9.3041)
+		(width 0.2)
+		(layer "B.Cu")
+		(net 5)
+	)
+	(segment
+		(start 54.3179 15.0155)
+		(end 51.0082 11.7058)
+		(width 0.2)
+		(layer "B.Cu")
+		(net 5)
+	)
+	(segment
+		(start 39.5301 9.3041)
+		(end 36.4379 9.3041)
+		(width 0.2)
+		(layer "B.Cu")
+		(net 5)
+	)
+	(segment
+		(start 51.0082 11.7058)
+		(end 41.9318 11.7058)
+		(width 0.2)
+		(layer "B.Cu")
+		(net 5)
+	)
+	(segment
+		(start 52.364 29.21)
+		(end 54.3179 27.2561)
+		(width 0.2)
+		(layer "B.Cu")
+		(net 5)
 	)
 	(segment
@@
 	)
 	(segment
-		(start 27.432 15.24)
-		(end 28.5337 15.24)
-		(width 0.2)
-		(layer "B.Cu")
-		(net 5)
-	)
-	(segment
-		(start 31.518 14.224)
-		(end 29.5497 14.224)
-		(width 0.2)
-		(layer "B.Cu")
-		(net 5)
-	)
-	(segment
-		(start 51.0082 11.7058)
-		(end 41.6998 11.7058)
-		(width 0.2)
-		(layer "B.Cu")
-		(net 5)
-	)
-	(segment
-		(start 29.5497 14.224)
-		(end 28.5337 15.24)
-		(width 0.2)
-		(layer "B.Cu")
-		(net 5)
-	)
-	(segment
-		(start 54.3179 15.0155)
-		(end 51.0082 11.7058)
-		(width 0.2)
-		(layer "B.Cu")
-		(net 5)
-	)
-	(segment
-		(start 39.2981 9.3041)
-		(end 36.4379 9.3041)
-		(width 0.2)
-		(layer "B.Cu")
-		(net 5)
-	)
-	(segment
-		(start 36.4379 9.3041)
-		(end 31.518 14.224)
-		(width 0.2)
-		(layer "B.Cu")
-		(net 5)
-	)
-	(segment
-		(start 41.6998 11.7058)
-		(end 39.2981 9.3041)
-		(width 0.2)
-		(layer "B.Cu")
-		(net 5)
-	)
-	(segment
-		(start 52.364 29.21)
-		(end 54.3179 27.2561)
-		(width 0.2)
-		(layer "B.Cu")
-		(net 5)
-	)
-	(segment
 		(start 8.885 31.1414)
 		(end 8.885 34.036)
@@
 	)
 	(segment
+		(start 44.45 35.306)
+		(end 43.18 34.036)
+		(width 0.2)
+		(layer "B.Cu")
+		(net 14)
+	)
+	(segment
 		(start 52.382 24.79)
-		(end 43.3509 24.79)
-		(width 0.2)
-		(layer "B.Cu")
-		(net 14)
-	)
-	(segment
-		(start 44.45 35.306)
-		(end 43.2594 34.1154)
-		(width 0.2)
-		(layer "B.Cu")
-		(net 14)
-	)
-	(segment
-		(start 43.3509 14.7821)
-		(end 38.9828 10.414)
-		(width 0.2)
-		(layer "B.Cu")
-		(net 14)
-	)
-	(segment
-		(start 43.2594 34.1154)
-		(end 43.2594 29.1658)
-		(width 0.2)
-		(layer "B.Cu")
-		(net 14)
-	)
-	(segment
-		(start 43.3509 29.0743)
-		(end 43.3509 24.79)
+		(end 44.552 24.79)
+		(width 0.2)
+		(layer "B.Cu")
+		(net 14)
+	)
+	(segment
+		(start 44.45 15.494)
+		(end 39.37 10.414)
+		(width 0.2)
+		(layer "B.Cu")
+		(net 14)
+	)
+	(segment
+		(start 44.45 24.892)
+		(end 44.45 15.494)
+		(width 0.2)
+		(layer "B.Cu")
+		(net 14)
+	)
+	(segment
+		(start 43.18 26.162)
+		(end 44.45 24.892)
+		(width 0.2)
+		(layer "B.Cu")
+		(net 14)
+	)
+	(segment
+		(start 43.18 34.036)
+		(end 43.18 26.162)
+		(width 0.2)
+		(layer "B.Cu")
+		(net 14)
+	)
+	(segment
+		(start 39.37 10.414)
+		(end 38.608 10.414)
 		(width 0.2)
 		(layer "B.Cu")
@@
 	)
 	(segment
-		(start 43.3509 24.79)
-		(end 43.3509 14.7821)
-		(width 0.2)
-		(layer "B.Cu")
-		(net 14)
-	)
-	(segment
-		(start 43.2594 29.1658)
-		(end 43.3509 29.0743)
-		(width 0.2)
-		(layer "B.Cu")
+		(start 44.552 24.79)
+		(end 44.45 24.892)
+		(width 0.2)
+		(layer "B.Cu")
